File: electrical/lcu03/lcu03.kicad_pcb (KiCad board)
At the start: 2 copper layers, 125 x 50 mm, 117 parts, among them P1 screw, P10 swd, P11 stepper_conn, P12 stepper_conn, P13 stepper_conn, P14 stepper_conn, P15 stepper_conn, P2 screw, P3 screw, P4 screw, P5 ext-1, P6 ~rst~, P7 mode, P8 ext-2, P9 USB_B, Q1 bc857, Q2 bc847, Q3 bc857, Q4 ntd18n06l, U1 crystal-4pin, U2 CP2102, U3 m24c02, U4 NCP3063, U5 MCP1703T-3302E/CB, U6 ts881, U7 lb1930mc, U8 a4985, U9 a4985

Commit message: a
Parts:
- moved P14 401.7 mm to (281.2, 54.2), turned to 90 degrees
- moved C27 348.9 mm to (256.2, 56.4), turned to 180 degrees
- moved C28 330.5 mm to (258.8, 49.3), turned to 270 degrees
- moved P13 329.5 mm to (206.3, 55.3), turned to 270 degrees
- moved R40 328.7 mm to (270.1, 55.1), turned to 180 degrees
- moved U8 327.1 mm to (263.6, 54.1)
- moved C32 316.1 mm to (271.0, 56.7)
- moved C29 315.7 mm to (257.3, 49.3), turned to 90 degrees
- moved R39 315.1 mm to (270.1, 52.9), turned to 180 degrees
- moved P11 310.2 mm to (208.7, 78.1), turned to 270 degrees
- moved C31 305.5 mm to (271.0, 51.3)
- moved C30 303.5 mm to (256.2, 52.3), turned to 180 degrees
- moved P12 289.1 mm to (206.2, 38.4), turned to 270 degrees
- moved C26 268.3 mm to (200.4, 73.2)
- moved D2 267.2 mm to (139.6, 118.2)
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
Commit message: a
Parts:
- removed C17: 680u, Capacitors_ThroughHole:C_Radial_D10_L20_P5
- added R45: 100 5%, Resistors_SMD:R_0805, F.Cu at (256.7, 55.3)
- added R46: 100 5%, Resistors_SMD:R_0805, F.Cu at (257.2, 85.4)
- moved P15 424.0 mm to (277.2, 84.2), turned to 270 degrees
- moved C38 374.3 mm to (270.6, 81.3)
- moved C22 355.8 mm to (260.5, 41.6)
- moved C37 355.4 mm to (261.8, 89.4)
- moved C34 351.9 mm to (259.0, 79.3), turned to 270 degrees
- moved U9 333.9 mm to (263.8, 84.2)
- moved R43 333.3 mm to (270.4, 82.8), turned to 180 degrees
- moved R44 328.8 mm to (270.4, 85.6), turned to 180 degrees
- moved R28 325.3 mm to (237.8, 70.1)
- moved C33 321.0 mm to (257.2, 87.4), turned to 180 degrees
- moved C36 317.4 mm to (257.3, 82.2), turned to 180 degrees
- moved P1 311.9 mm to (209.6, 74.5)
- moved C35 305.5 mm to (257.5, 78.3), turned to 90 degrees
- moved R29 298.3 mm to (241.6, 70.0)
- moved R30 295.2 mm to (238.3, 66.3)
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Connections:
- C31 pad 1: /stepper-subcircuit-1/Vbb -> /stepper-subcircuit-1/ref
- C37 pad 1: /stepper-subcircuit-1/Vbb -> /stepper-subcircuit-1/ref
- P14 pad 1: /stepper-subcircuit-1/out1a-1 -> /stepper-subcircuit-1/out2b-1
- P14 pad 2: /stepper-subcircuit-1/out1b-1 -> /stepper-subcircuit-1/out2a-1
- P14 pad 3: /stepper-subcircuit-1/out2a-1 -> /stepper-subcircuit-1/out1a-1
- P14 pad 4: /stepper-subcircuit-1/out2b-1 -> /stepper-subcircuit-1/out1b-1
- P15 pad 1: /stepper-subcircuit-2/out1a-1 -> /stepper-subcircuit-2/out2b-1
- P15 pad 2: /stepper-subcircuit-2/out1b-1 -> /stepper-subcircuit-2/out2a-1
- P15 pad 3: /stepper-subcircuit-2/out2a-1 -> /stepper-subcircuit-2/out1a-1
- P15 pad 4: /stepper-subcircuit-2/out2b-1 -> /stepper-subcircuit-2/out1b-1
- U8 pad 8: GND -> Net-(R45-Pad2)
- U9 pad 8: GND -> Net-(R46-Pad2)
Routing:
- net GND: track 0.00 -> 69.5 mm, vias 0 -> 4
- net /stepper-subcircuit-1/Vbb: track 0.00 -> 19.7 mm, vias 0 -> 2
- net /stepper-subcircuit-1/~reset~: track 0.00 -> 12.5 mm
- net /stepper-subcircuit-1/~sleep~: track 0.00 -> 12.5 mm
- net /stepper-subcircuit-1/ms1: track 0.00 -> 12.3 mm
- net /stepper-subcircuit-1/ms2: track 0.00 -> 12.2 mm
- net /stepper-subcircuit-1/out2b-1: track 0.00 -> 11.4 mm
- net /shutter-out-b: track 0.00 -> 11.0 mm
- net /stepper-subcircuit-2/out2b-1: track 0.00 -> 10.7 mm
- net /stepper-subcircuit-1/out1b-1: track 0.00 -> 10.7 mm
- net /stepper-subcircuit-1/out2a-1: track 0.00 -> 10.1 mm
- net /stepper-subcircuit-1/out1a-1: track 0.00 -> 10.1 mm
- net /stepper-subcircuit-2/out1b-1: track 0.00 -> 9.94 mm
- net /stepper-subcircuit-2/out2a-1: track 0.00 -> 9.50 mm
- net /stepper-subcircuit-2/out1a-1: track 0.00 -> 9.50 mm
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
Commit message: a
Parts:
- moved C2 121.7 mm to (41.4, 166.6), turned to 90 degrees
- moved P6 119.9 mm to (50.6, 165.5), turned to 270 degrees
- moved C3 117.0 mm to (47.1, 164.1), turned to 270 degrees
- moved U1 116.2 mm to (43.2, 162.9), turned to 180 degrees
- moved R8 116.2 mm to (51.4, 162.9), turned to 270 degrees
- moved C4 115.0 mm to (49.8, 162.8), turned to 90 degrees
- moved C23 114.8 mm to (98.7, 154.0)
- moved R17 114.8 mm to (96.1, 156.6)
- moved R18 114.8 mm to (96.3, 159.1)
- moved R21 114.8 mm to (101.3, 156.6)
- moved R22 114.8 mm to (99.2, 159.1)
- moved U6 114.8 mm to (98.7, 156.6)
- moved R6 108.6 mm to (44.2, 157.7), turned to 270 degrees
- moved C11 108.2 mm to (46.5, 157.7), turned to 270 degrees
- moved C8 105.7 mm to (39.8, 154.8), turned to 270 degrees
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Routing:
- net VDD: track 6.21 -> 78.5 mm
- net GND: track 69.5 -> 126.3 mm
- net Net-(D4-Pad2): track 0.00 -> 23.8 mm
- net Net-(L2-Pad1): track 0.00 -> 21.9 mm
- net /clk-in: track 0.00 -> 13.9 mm
- net /reg-fb: track 0.00 -> 13.9 mm
- net Net-(C20-Pad1): track 0.00 -> 13.6 mm
- net /~mcu-rst~: track 0.00 -> 12.6 mm
- net Net-(Q2-Pad2): track 0.00 -> 10.2 mm
- net /d+: track 0.00 -> 9.77 mm
- net /d-: track 0.00 -> 6.85 mm
- net Net-(C3-Pad1): track 0.00 -> 6.18 mm
- net /suspend: track 0.00 -> 5.55 mm
- net Net-(C16-Pad2): track 0.00 -> 5.41 mm
- net /Vbus: track 0.00 -> 5.27 mm
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
Commit message: a
Parts:
- R12: footprint Resistors_SMD:R_0805 -> Capacitors_SMD:C_1206
- moved P12 144.9 mm to (138.6, 108.4), turned to 180 degrees
- moved P13 140.4 mm to (138.6, 75.3), turned to 0 degrees
- moved R34 139.9 mm to (136.6, 103.5)
- moved R33 136.6 mm to (140.6, 103.5), turned to 0 degrees
- moved R35 136.1 mm to (136.6, 80.2)
- moved R36 132.4 mm to (140.6, 80.2), turned to 0 degrees
- moved P15 121.7 mm to (160.6, 118.9), turned to 180 degrees
- moved C32 118.7 mm to (156.1, 80.6), turned to 180 degrees
- moved P14 118.5 mm to (160.8, 74.3), turned to 0 degrees
- moved R26 116.7 mm to (128.6, 77.4)
- moved R23 116.7 mm to (125.7, 77.4)
- moved R27 116.7 mm to (126.2, 79.0)
- moved R39 116.1 mm to (158.0, 79.1), turned to 0 degrees
- moved R44 114.3 mm to (159.2, 112.1), turned to 90 degrees
- moved R19 113.1 mm to (122.6, 74.9)
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Routing:
- net GND: track 126.3 -> 238.7 mm, vias 4 -> 2
- net /Vbus: track 5.27 -> 67.4 mm, vias 0 -> 1
- net VDD: track 78.5 -> 126.8 mm
- net Net-(D4-Pad2): track 23.8 -> 56.4 mm
- net Net-(C20-Pad1): track 13.6 -> 28.4 mm
- net Net-(C18-Pad1): track 0.00 -> 10.9 mm
- net Net-(P11-Pad1): track 8.71 -> 18.8 mm
- net /shutter-out-b: track 11.0 -> 21.0 mm
- net /hall2: track 0.00 -> 7.58 mm
- net /stepper-subcircuit-1/out1b-1: track 10.7 -> 3.21 mm
- net /hall1: track 0.00 -> 7.21 mm
- net /stepper-subcircuit-1/out2b-1: track 11.4 -> 6.28 mm
- net Net-(D3-Pad2): track 0.00 -> 4.63 mm
- net Net-(Q1-Pad3): track 0.00 -> 4.31 mm
- net Net-(P13-Pad3): track 0.00 -> 3.80 mm
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
Commit message: a
Parts:
- added P16: screw, Mounting_Holes:MountingHole_3mm, F.Cu at (161.5, 74.5)
- added P17: screw, Mounting_Holes:MountingHole_3mm, F.Cu at (161.5, 117.5)
- moved Q4 36.6 mm to (170.4, 117.7), turned to 0 degrees
- moved Q2 33.0 mm to (177.1, 117.3), turned to 90 degrees
- moved Q3 32.9 mm to (177.1, 114.0)
- moved L2 30.4 mm to (171.5, 87.0)
- moved C24 29.9 mm to (180.0, 98.8)
- moved D4 27.8 mm to (178.5, 94.0)
- moved C13 27.1 mm to (174.8, 94.5)
- moved C15 27.1 mm to (174.8, 96.0)
- moved C19 27.1 mm to (174.7, 105.0)
- moved C20 27.1 mm to (170.7, 105.8)
- moved R24 27.1 mm to (172.2, 105.8)
- moved R25 27.1 mm to (174.3, 106.7)
- moved U4 27.1 mm to (172.8, 100.7)
- moved C16 27.1 mm to (177.6, 101.3)
- moved R12 27.1 mm to (171.8, 94.8)
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Routing:
- net /reg-fb: track 13.9 -> 33.3 mm
- net /Vbus: track 67.4 -> 55.0 mm
- net /stepper-subcircuit-1/out2b-1: track 6.28 -> 18.5 mm
- net /stepper-subcircuit-1/out1b-1: track 3.21 -> 12.4 mm
- net Net-(Q2-Pad2): track 10.2 -> 19.0 mm
- net Net-(C20-Pad1): track 28.4 -> 37.0 mm
- net /stepper-subcircuit-1/ms2: track 12.2 -> 4.36 mm
- net /stepper-subcircuit-1/~reset~: track 12.5 -> 5.90 mm
- net /stepper-subcircuit-1/ms1: track 12.3 -> 6.04 mm
- net Net-(D4-Pad2): track 56.4 -> 50.3 mm
- net GND: track 238.7 -> 243.5 mm, vias 2 -> 3
- net Net-(Q1-Pad3): track 4.31 -> 0.00 mm
- net /stepper-subcircuit-1/ref: track 9.59 -> 6.17 mm
- net VDD: track 126.8 -> 129.1 mm
- net /stepper-subcircuit-1/Vbb: track 19.9 -> 22.1 mm, vias 1 -> 3
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Other:
- board size 125 x 50 mm -> 99.5 x 50 mm

Commit message: a
Parts:
- moved R38 2.14 mm to (129.4, 90.7), turned to 0 degrees
- moved C38 2.06 mm to (156.8, 109.3), turned to 0 degrees
- moved R41 1.69 mm to (132.4, 91.5), turned to 0 degrees
- moved R7 1.45 mm to (135.6, 93.7)
- moved R43 1.15 mm to (154.3, 110.7)
- moved R44 0.21 mm to (150.4, 110.0)
Routing:
- net GND: track 243.5 -> 270.2 mm
- net VDD: track 129.1 -> 141.4 mm
- net /swd-clk: track 0.00 -> 7.65 mm
- net /stepper-subcircuit-2/step: track 3.21 -> 9.60 mm
- net /stepper-subcircuit-2/out2b-1: track 10.7 -> 15.5 mm
- net /swd-io: track 0.00 -> 4.26 mm
- net /stepper-subcircuit-1/ms2: track 4.36 -> 8.12 mm
- net /stepper-subcircuit-1/dir: track 3.46 -> 7.07 mm
- net /stepper-subcircuit-1/Vbb: track 22.1 -> 25.5 mm, vias 3 -> 5
- net /stepper-subcircuit-1/ms1: track 6.04 -> 8.74 mm
- net /stepper-subcircuit-2/out2a-1: track 9.50 -> 12.1 mm
- net /stepper-subcircuit-2/out1b-1: track 9.94 -> 11.8 mm
- net /stepper-subcircuit-1/~reset~: track 5.90 -> 7.36 mm
- net /stepper-subcircuit-2/rsense2-1: track 2.78 -> 3.82 mm
- net /stepper-subcircuit-2/dir: track 4.27 -> 3.33 mm

Commit message: a
Parts:
- added R47: 10k 5%, Resistors_SMD:R_0805, F.Cu at (105.2, 81.5)
- moved R37 19.8 mm to (131.7, 94.0), turned to 180 degrees
- moved R42 15.3 mm to (132.6, 97.7), turned to 180 degrees
- moved R41 9.38 mm to (129.8, 100.5), turned to 180 degrees
- moved R7 0.85 mm to (135.6, 92.8)
Connections:
- net /stepper-subcircuit-1/out1a-1 renamed /stepper-subcircuit-1/out1a
- net /stepper-subcircuit-1/out1b-1 renamed /stepper-subcircuit-1/out1b
- net /stepper-subcircuit-1/out2a-1 renamed /stepper-subcircuit-1/out2a
- net /stepper-subcircuit-1/out2b-1 renamed /stepper-subcircuit-1/out2b
- net /stepper-subcircuit-1/rsense1-1 renamed /stepper-subcircuit-1/rsense1
- net /stepper-subcircuit-1/rsense2-1 renamed /stepper-subcircuit-1/rsense2
- net /stepper-subcircuit-2/out1a-1 renamed /stepper-subcircuit-2/out1a
- net /stepper-subcircuit-2/out1b-1 renamed /stepper-subcircuit-2/out1b
- net /stepper-subcircuit-2/out2a-1 renamed /stepper-subcircuit-2/out2a
- net /stepper-subcircuit-2/out2b-1 renamed /stepper-subcircuit-2/out2b
- net /stepper-subcircuit-2/rsense1-1 renamed /stepper-subcircuit-2/rsense1
- net /stepper-subcircuit-2/rsense2-1 renamed /stepper-subcircuit-2/rsense2
- R37 pad 1: /stepper-subcircuit-1/step -> Net-(R37-Pad1)
- R38 pad 1: /stepper-subcircuit-1/dir -> Net-(R38-Pad1)
- R41 pad 1: /stepper-subcircuit-2/step -> Net-(R41-Pad1)
- R42 pad 1: /stepper-subcircuit-2/dir -> Net-(R42-Pad1)
- U8 pad 11: /stepper-subcircuit-1/step -> Net-(R37-Pad1)
- U8 pad 14: /stepper-subcircuit-1/dir -> Net-(R38-Pad1)
- U9 pad 11: /stepper-subcircuit-2/step -> Net-(R41-Pad1)
- U9 pad 14: /stepper-subcircuit-2/dir -> Net-(R42-Pad1)
- stm1 pad 11: /shutter-b -> /stepper-subcircuit-2/step
- stm1 pad 14: /stepper-subcircuit-1/~enable~ -> /stepper-subcircuit-2/dir
- stm1 pad 18: /gpio-3 -> /stepper-subcircuit-1/step
- stm1 pad 19: /~wc~ -> /shutter-b
- stm1 pad 21: /stepper-subcircuit-2/step -> /stepper-subcircuit-1/~enable~
- stm1 pad 25: /stepper-subcircuit-2/dir -> /gpio-3
- stm1 pad 29: /suspend -> /gpio-2
- stm1 pad 41: /gpio-2 -> /suspend
- stm1 pad 46: /stepper-subcircuit-1/step -> /~wc~
Routing:
- net /stepper-subcircuit-1/~enable~: track 7.16 -> 33.9 mm
- net /rxd: track 0.00 -> 26.7 mm
- net /txd: track 0.00 -> 25.2 mm, vias 0 -> 2
- net /i2c1-scl: track 0.00 -> 22.7 mm, vias 0 -> 2
- net /i2c1-sda: track 0.00 -> 22.6 mm, vias 0 -> 2
- net /rts: track 0.00 -> 22.3 mm
- net /cts: track 0.00 -> 20.3 mm
- net /~wc~: track 1.75 -> 20.9 mm, vias 0 -> 2
- net /boot0: track 0.00 -> 14.1 mm, vias 0 -> 2
- net /boot1: track 0.00 -> 9.82 mm
- net VDD: track 141.4 -> 150.2 mm
- net GND: track 270.2 -> 278.8 mm
- net /suspend: track 5.55 -> 13.0 mm
- net Net-(R38-Pad1): track 0.00 -> 4.96 mm
- net /stepper-subcircuit-1/dir: track 7.07 -> 2.11 mm
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
Commit message: a
Parts:
- moved Q2 1.78 mm to (178.2, 118.7)
- moved Q3 1.78 mm to (178.2, 115.4)
- moved R17 0.45 mm to (95.0, 109.2)
Connections:
- stm1 pad 15: /stepper-subcircuit-1/~reset~ -> /hall1
- stm1 pad 19: /shutter-b -> /gpio-0
- stm1 pad 26: /hall1 -> /stepper-subcircuit-1/~reset~
- stm1 pad 28: /ext-power-flag -> /gpio-1
- stm1 pad 4: /gpio-0 -> /shutter-b
- stm1 pad 45: /gpio-1 -> /ext-power-flag
Routing:
- net GND: track 278.8 -> 365.4 mm, vias 3 -> 5
- net /led-0: track 0.00 -> 39.3 mm, vias 0 -> 2
- net /led-1: track 0.00 -> 37.9 mm, vias 0 -> 2
- net /reg-fb: track 33.3 -> 69.4 mm, vias 0 -> 1
- net /ext-power-flag: track 0.00 -> 33.4 mm, vias 0 -> 2
- net /shutter-a: track 0.00 -> 30.8 mm
- net /shutter-b: track 0.00 -> 26.0 mm
- net /stepper-subcircuit-1/~sleep~: track 13.1 -> 36.9 mm
- net Net-(R42-Pad1): track 3.33 -> 22.5 mm
- net Net-(R41-Pad1): track 3.21 -> 20.8 mm, vias 0 -> 2
- net /hall1: track 7.21 -> 24.1 mm
- net /stepper-subcircuit-1/Vbb: track 25.5 -> 32.4 mm, vias 5 -> 6
- net Net-(C3-Pad1): track 6.18 -> 11.4 mm
- net /tx-2: track 0.00 -> 4.43 mm
- net /rx-2: track 0.00 -> 3.69 mm
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