File: electrical/lcu03/lcu03.kicad_pcb (KiCad board)
At the start: 2 copper layers, 99.5 x 50 mm, 121 parts, among them P1 screw, P10 swd, P11 stepper_conn, P12 stepper_conn, P13 stepper_conn, P14 stepper_conn, P15 stepper_conn, P16 screw, P17 screw, P2 screw, P3 screw, P4 screw, P5 ext-1, P6 ~rst~, P7 mode, P8 ext-2, P9 USB_B, Q1 bc857, Q2 bc847, Q3 bc857, Q4 ntd18n06l, U1 crystal-4pin, U2 CP2102, U3 m24c02, U4 NCP3063, U5 MCP1703T-3302E/CB, U6 ts881, U7 lb1930mc, U8 a4985, U9 a4985

Commit message: a
Parts:
- moved P5 45.5 mm to (100.5, 119.0)
- moved P8 45.5 mm to (100.5, 73.0)
- moved R4 40.7 mm to (117.2, 115.2), turned to 270 degrees
- moved R10 39.6 mm to (105.6, 116.5), turned to 180 degrees
- moved R11 39.6 mm to (108.6, 116.5), turned to 0 degrees
Connections:
- P5 pad 1: /tx-2 -> /Vbus
- P5 pad 2: /rx-2 -> GND
- P5 pad 3: GND -> /i2c1-scl
- P5 pad 4: /i2c1-scl -> /i2c1-sda
- P5 pad 5: /i2c1-sda -> GND
- P5 pad 6: GND -> /tx-2
- P5 pad 7: /Vbus -> /rx-2
Routing:
- net GND: track 365.4 -> 424.4 mm, vias 5 -> 7
- net /stepper-subcircuit-1/Vbb: track 32.4 -> 66.6 mm
- net /rx-2: track 3.69 -> 37.7 mm, vias 0 -> 2
- net /tx-2: track 4.43 -> 38.3 mm, vias 0 -> 2
- net /i2c1-scl: track 22.7 -> 45.2 mm, vias 2 -> 3
- net /i2c1-sda: track 22.6 -> 42.4 mm, vias 2 -> 3
- net VDD: track 149.9 -> 165.9 mm
- net /reg-fb: track 69.4 -> 57.5 mm
- net /Vbus: track 57.9 -> 65.0 mm
- net /hall2: track 7.58 -> 8.84 mm

Commit message: a
Parts:
- moved D4 4.00 mm to (182.4, 93.1)
- moved L2 3.40 mm to (174.9, 87.1)
- turned R38 to 180 degrees
Connections:
- stm1 pad 17: /~high-current~ -> /stepper-subcircuit-1/~reset~
- stm1 pad 25: /gpio-3 -> /hall2
- stm1 pad 26: /stepper-subcircuit-1/~reset~ -> /~high-current~
- stm1 pad 27: /hall2 -> /gpio-3
Routing:
- net GND: track 424.4 -> 657.3 mm, vias 7 -> 13
- net /reg-fb: track 57.5 -> 143.7 mm, vias 1 -> 2
- net /stepper-subcircuit-1/ref: track 6.17 -> 74.5 mm, vias 0 -> 3
- net /stepper-subcircuit-1/Vbb: track 66.6 -> 115.3 mm, vias 6 -> 8
- net Net-(R38-Pad1): track 4.96 -> 45.6 mm, vias 0 -> 2
- net /stepper-subcircuit-1/~reset~: track 7.36 -> 38.1 mm
- net /stepper-subcircuit-1/ms2: track 8.12 -> 34.4 mm, vias 0 -> 4
- net /stepper-subcircuit-1/ms1: track 8.74 -> 32.7 mm, vias 0 -> 4
- net /~high-current~: track 1.90 -> 20.3 mm
- net /hall2: track 8.84 -> 25.1 mm
- net /stepper-subcircuit-1/~sleep~: track 36.9 -> 48.1 mm, vias 0 -> 2
- net VDD: track 165.9 -> 174.9 mm, vias 0 -> 1
- net Net-(Q1-Pad3): track 0.00 -> 2.11 mm
- net /stepper-subcircuit-1/dir: track 2.11 -> 3.61 mm
- net /stepper-subcircuit-1/~enable~: track 34.1 -> 32.7 mm
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
Commit message: a
Routing:
- net GND: track 657.3 -> 769.3 mm, vias 13 -> 17
- net /Vbus: track 65.0 -> 174.4 mm, vias 2 -> 3
- net Net-(R37-Pad1): track 4.01 -> 35.0 mm, vias 0 -> 2
- net /led-1: track 37.8 -> 42.5 mm
- net /led-0: track 39.3 -> 43.9 mm
- net /ext-power-flag: track 33.4 -> 37.2 mm
- net /stepper-subcircuit-1/~sleep~: track 48.1 -> 46.4 mm
- net /reg-fb: track 143.7 -> 142.5 mm
- net /stepper-subcircuit-1/ref: track 74.5 -> 75.4 mm
- net Net-(R38-Pad1): track 45.6 -> 44.8 mm
- net /rx-2: track 37.7 -> 37.1 mm
- net /stepper-subcircuit-1/Vbb: track 115.3 -> 115.8 mm

Commit message: a
Parts:
- moved C37 1.45 mm to (146.8, 102.8)
- moved C4 0.59 mm to (126.0, 106.7)
Routing:
- net VDD: track 174.9 -> 371.2 mm, vias 1 -> 11
- net /Vbus: track 174.4 -> 266.3 mm, vias 3 -> 5
- net /stepper-subcircuit-1/Vbb: track 115.8 -> 184.9 mm, vias 8 -> 9
- net /reg-fb: track 142.5 -> 210.2 mm, vias 2 -> 3
- net GND: track 769.3 -> 831.7 mm, vias 17 -> 18
- net /stepper-subcircuit-1/~enable~: track 32.7 -> 91.8 mm, vias 0 -> 2
- net /gpio-0: track 0.00 -> 31.7 mm, vias 0 -> 6
- net /gpio-2: track 0.00 -> 21.5 mm
- net /gpio-1: track 0.00 -> 19.5 mm
- net /gpio-3: track 0.00 -> 17.9 mm
- net /stepper-subcircuit-1/ref: track 75.4 -> 80.7 mm
- net /stepper-subcircuit-2/out2b: track 15.5 -> 20.2 mm
- net /hall2: track 25.1 -> 28.6 mm
- net /~mcu-rst~: track 15.9 -> 17.6 mm
- net Net-(R41-Pad1): track 20.8 -> 22.4 mm
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
Commit message: Finished routing.
Connections:
- stm1 pad 19: /gpio-0 -> /gpio-3
- stm1 pad 27: /gpio-3 -> /gpio-2
- stm1 pad 29: /gpio-2 -> /gpio-0
Routing:
- net /gpio-3: track 17.9 -> 34.6 mm, vias 0 -> 6
- net /stepper-subcircuit-1/Vbb: track 184.9 -> 180.1 mm
- net /gpio-0: track 31.7 -> 27.1 mm, vias 6 -> 0
- net /gpio-1: track 19.5 -> 22.8 mm
- net Net-(D2-Pad1): track 0.00 -> 1.65 mm
- net Net-(D1-Pad1): track 0.00 -> 1.65 mm
- net GND: track 831.7 -> 832.3 mm
- added copper zone on B.Cu, net GND
- added copper zone on F.Cu, net GND
- added copper zone on F.Cu, net Net-(D4-Pad2)

Commit message: Generated drill and fabrication files.
Routing:
- net VDD: track 371.5 -> 373.9 mm
- net GND: track 832.3 -> 834.7 mm
- net /stepper-subcircuit-1/~sleep~: track 46.4 -> 44.6 mm

Commit message: Included fixtures in User comments layer.
Other:
- board text added: "Here make just short circuit."
- board text added: "Here use 2n4 instead to decrease frequency down to 150kHz."
- board text added: "Mot use it. Use through hole 8.2Ohm instead."
- board text added: "Use two pullup 0Ohm to make step/8."
Changed lines of the file:
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@@
     (area 80.524999 62.15 204.999999 123.47626)
     (thickness 1.6)
-    (drawings 7)
+    (drawings 47)
     (tracks 2016)
     (zones 0)
@@
   (layers
     (0 F.Cu signal)
-    (31 B.Cu signal)
+    (31 B.Cu signal hide)
     (34 B.Paste user)
     (35 F.Paste user)
@@
   )
   (setup
-    (last_trace_width 0.4)
+    (last_trace_width 0.25)
     (user_trace_width 0.4)
     (user_trace_width 0.6)
@@
     )
   )
+  (gr_text "Use two pullup \n0Ohm to make step/8." (at 135.5 84) (layer Dwgs.User)
+    (effects (font (size 0.5 0.5) (thickness 0.125)))
+  )
+  (gr_line (start 136.5 87) (end 133.5 90) (angle 90) (layer Dwgs.User) (width 0.2))
+  (gr_line (start 133.5 87) (end 136.5 90) (angle 90) (layer Dwgs.User) (width 0.2))
+  (gr_line (start 132.5 87) (end 133 87) (angle 90) (layer Dwgs.User) (width 0.2))
+  (gr_line (start 132.5 90) (end 132.5 87) (angle 90) (layer Dwgs.User) (width 0.2))
+  (gr_line (start 137.5 90) (end 132.5 90) (angle 90) (layer Dwgs.User) (width 0.2))
+  (gr_line (start 137.5 87) (end 137.5 90) (angle 90) (layer Dwgs.User) (width 0.2))
+  (gr_line (start 133 87) (end 137.5 87) (angle 90) (layer Dwgs.User) (width 0.2))
+  (gr_line (start 108 113) (end 105.5 115.5) (angle 90) (layer Dwgs.User) (width 0.2))
+  (gr_line (start 105.5 113) (end 108 115.5) (angle 90) (layer Dwgs.User) (width 0.2))
+  (gr_line (start 108.5 113) (end 105 113) (angle 90) (layer Dwgs.User) (width 0.2))
+  (gr_line (start 108.5 115.5) (end 108.5 113) (angle 90) (layer Dwgs.User) (width 0.2))
+  (gr_line (start 105 115.5) (end 108.5 115.5) (angle 90) (layer Dwgs.User) (width 0.2))
+  (gr_line (start 105 113) (end 105 115.5) (angle 90) (layer Dwgs.User) (width 0.2))
+  (gr_text "Here use 2n4 instead \nto decrease frequency \ndown to 150kHz." (at 179.5 99) (layer Dwgs.User)
+    (effects (font (size 0.5 0.5) (thickness 0.125)))
+  )
+  (gr_line (start 176 104) (end 177 104) (angle 90) (layer Dwgs.User) (width 0.2))
+  (gr_line (start 176 104) (end 176 103) (angle 90) (layer Dwgs.User) (width 0.2))
+  (gr_line (start 176 104) (end 179.5 100.5) (angle 90) (layer Dwgs.User) (width 0.2))
+  (gr_line (start 139 111.5) (end 141.5 114) (angle 90) (layer Dwgs.User) (width 0.2))
+  (gr_line (start 135 111.5) (end 139 111.5) (angle 90) (layer Dwgs.User) (width 0.2))
+  (gr_line (start 131 115.5) (end 130 115.5) (angle 90) (layer Dwgs.User) (width 0.2))
+  (gr_line (start 132.5 114) (end 131 115.5) (angle 90) (layer Dwgs.User) (width 0.2))
+  (gr_line (start 134.5 111) (end 132 113.5) (angle 90) (layer Dwgs.User) (width 0.2))
+  (gr_line (start 135.5 112) (end 134.5 111) (angle 90) (layer Dwgs.User) (width 0.2))
+  (gr_line (start 133 114.5) (end 135.5 112) (angle 90) (layer Dwgs.User) (width 0.2))
+  (gr_line (start 132 113.5) (end 133 114.5) (angle 90) (layer Dwgs.User) (width 0.2))
+  (gr_text "Mot use it. Use through \nhole 8.2Ohm instead." (at 128.5 112) (layer Dwgs.User)
+    (effects (font (size 0.5 0.5) (thickness 0.125)))
+  )
+  (gr_text "Here make just \nshort circuit." (at 166.5 105) (layer Dwgs.User)
+    (effects (font (size 0.5 0.5) (thickness 0.125)))
+  )
+  (gr_line (start 173 104) (end 169.5 107.5) (angle 90) (layer Dwgs.User) (width 0.2))
+  (gr_line (start 169.5 104) (end 173 107.5) (angle 90) (layer Dwgs.User) (width 0.2))
+  (gr_line (start 169.5 107.5) (end 169.5 104) (angle 90) (layer Dwgs.User) (width 0.2))
+  (gr_line (start 173 107.5) (end 169.5 107.5) (angle 90) (layer Dwgs.User) (width 0.2))
+  (gr_line (start 173 104) (end 173 107.5) (angle 90) (layer Dwgs.User) (width 0.2))
+  (gr_line (start 169.5 104) (end 173 104) (angle 90) (layer Dwgs.User) (width 0.2))
+  (gr_line (start 130.5 114) (end 128.5 116) (angle 90) (layer Dwgs.User) (width 0.2))
+  (gr_line (start 128.5 114) (end 130.5 116) (angle 90) (layer Dwgs.User) (width 0.2))
+  (gr_line (start 130.5 113) (end 128.5 113) (angle 90) (layer Dwgs.User) (width 0.2))
+  (gr_line (start 130.5 116.5) (end 130.5 113) (angle 90) (layer Dwgs.User) (width 0.2))
+  (gr_line (start 128.5 116.5) (end 130.5 116.5) (angle 90) (layer Dwgs.User) (width 0.2))
+  (gr_line (start 128.5 113) (end 128.5 116.5) (angle 90) (layer Dwgs.User) (width 0.2))
   (dimension 99.5 (width 0.3) (layer Dwgs.User)
     (gr_text "99.500 mm" (at 137.75 63.65) (layer Dwgs.User)
