File: electrical/lcu03/lcu03.sch (KiCad schematic (older format))
At the start: 92 parts, among them P1 screw, P10 swd, P11 stepper_conn, P12 stepper_conn, P13 stepper_conn, P2 screw, P3 screw, P4 screw, P5 ext-1, P6 ~rst~, P7 mode, P8 ext-2, P9 USB_B, Q1 bc857, Q2 bc847, Q3 bc857, Q4 ntd18n06l, U1 crystal-4pin, U2 CP2102, U3 m24c02, U4 NCP3063, U5 MCP1703T-3302E/CB, U6 ts881, U7 lb1930mc

Commit message: a
Parts:
- R12: footprint Resistors_SMD:R_0805 -> Capacitors_SMD:C_1206

Commit message: a
Parts:
- added P16, P17: screw, Mounting_Holes:MountingHole_3mm, symbol TST
Connections:
- wire segments 365 -> 367

Commit message: a
Parts:
- added R47: 10k 5%, Resistors_SMD:R_0805, symbol R
Connections:
- wire segments 367 -> 369

Commit message: a
Changed lines of the file:
@@
 Text Label 9800 3200 0    60   ~ 0
 rx-2
-Text Label 4150 6600 0    60   ~ 0
+Text Label 9250 7150 0    60   ~ 0
 gpio-0
-Text Label 9700 8100 0    60   ~ 0
+Text Label 9700 9500 0    60   ~ 0
 gpio-1
 Text Label 9700 4200 0    60   ~ 0
@@
 	4550 5900 4100 5900
 Wire Wire Line
-	4550 6600 4100 6600
+	9600 7150 9150 7150
 Wire Wire Line
 	1200 12950 1200 12750
@@
 	9150 4200 10000 4200
 Wire Wire Line
-	9150 8100 10000 8100
+	9150 9500 10000 9500
 Wire Wire Line
 	2600 12650 3550 12650
@@
 Text Label 9200 2600 0    60   ~ 0
 shutter-a
-Text Label 9200 7150 0    60   ~ 0
+Text Label 4100 6600 0    60   ~ 0
 shutter-b
 Text Label 9200 8500 0    60   ~ 0
 ~enable~
-Text Label 9200 3600 0    60   ~ 0
+Text Label 9200 9100 0    60   ~ 0
 ~reset~
 Text Label 9200 3800 0    60   ~ 0
@@
 Text Label 9200 3400 0    60   ~ 0
 dir2
-Text Label 9200 9100 0    60   ~ 0
+Text Label 9200 3600 0    60   ~ 0
 hall1
 Text Label 9200 9300 0    60   ~ 0
 hall2
-Text Label 9200 9500 0    60   ~ 0
+Text Label 9200 8100 0    60   ~ 0
 ext-power-flag
 Wire Wire Line
 	9150 2600 9650 2600
 Wire Wire Line
-	9150 7150 9650 7150
+	4050 6600 4550 6600
 Wire Wire Line
 	9150 8500 9500 8500
 Wire Wire Line
-	9150 3600 9500 3600
+	9150 9100 9500 9100
 Wire Wire Line
 	9150 3800 9500 3800
@@
 	9150 3400 9450 3400
 Wire Wire Line
-	9150 9100 9450 9100
+	9150 3600 9450 3600
 Wire Wire Line
 	9150 9300 9450 9300
 Wire Wire Line
-	9150 9500 9950 9500
+	9150 8100 9950 8100
 $Comp
 L m24c02 U3

Commit message: a
Connections:
- wire segments 369 -> 371
Other:
- moved on the sheet: R4
Changed lines of the file:
@@
 Text Label 9700 8900 0    60   ~ 0
 gpio-3
-Text Label 2700 12550 0    60   ~ 0
+Text Label 2700 13050 0    60   ~ 0
 tx-2
-Text Label 2700 12650 0    60   ~ 0
+Text Label 2700 13150 0    60   ~ 0
 rx-2
 $Comp
 L R R4
 U 1 1 56676C7C
-P 3550 12350
-F 0 "R4" V 3630 12350 50  0000 C CNN
-F 1 "10k 5%" V 3550 12350 50  0000 C CNN
-F 2 "Resistors_SMD:R_0805" V 3480 12350 30  0001 C CNN
-F 3 "" H 3550 12350 30  0000 C CNN
-	1    3550 12350
+P 3250 13550
+F 0 "R4" V 3330 13550 50  0000 C CNN
+F 1 "10k 5%" V 3250 13550 50  0000 C CNN
+F 2 "Resistors_SMD:R_0805" V 3180 13550 30  0001 C CNN
+F 3 "" H 3250 13550 30  0000 C CNN
+	1    3250 13550
 	1    0    0    -1
 $EndComp
@@
 L VDD #PWR030
 U 1 1 56676C7D
-P 3550 12100
-F 0 "#PWR030" H 3550 12200 30  0001 C CNN
-F 1 "VDD" H 3550 12210 30  0000 C CNN
-F 2 "" H 3550 12100 60  0000 C CNN
-F 3 "" H 3550 12100 60  0000 C CNN
-	1    3550 12100
-	1    0    0    -1
-$EndComp
+P 3250 13300
+F 0 "#PWR030" H 3250 13400 30  0001 C CNN
+F 1 "VDD" H 3250 13410 30  0000 C CNN
+F 2 "" H 3250 13300 60  0000 C CNN
+F 3 "" H 3250 13300 60  0000 C CNN
+	1    3250 13300
+	1    0    0    -1
+$EndComp
+Text Label 2700 12750 0    60   ~ 0
+i2c1-scl
 Text Label 2700 12850 0    60   ~ 0
-i2c1-scl
-Text Label 2700 12950 0    60   ~ 0
 i2c1-sda
 $Comp
 L GND #PWR031
 U 1 1 56676C7E
-P 3550 12850
-F 0 "#PWR031" H 3550 12600 50  0001 C CNN
-F 1 "GND" H 3550 12700 50  0000 C CNN
-F 2 "" H 3550 12850 60  0000 C CNN
-F 3 "" H 3550 12850 60  0000 C CNN
-	1    3550 12850
+P 3550 12750
+F 0 "#PWR031" H 3550 12500 50  0001 C CNN
+F 1 "GND" H 3550 12600 50  0000 C CNN
+F 2 "" H 3550 12750 60  0000 C CNN
+F 3 "" H 3550 12750 60  0000 C CNN
+	1    3550 12750
 	1    0    0    -1
 $EndComp
@@
 L GND #PWR032
 U 1 1 56676C7F
-P 3550 13150
-F 0 "#PWR032" H 3550 12900 50  0001 C CNN
-F 1 "GND" H 3550 13000 50  0000 C CNN
-F 2 "" H 3550 13150 60  0000 C CNN
-F 3 "" H 3550 13150 60  0000 C CNN
-	1    3550 13150
-	1    0    0    -1
-$EndComp
-Text Label 2950 13150 0    60   ~ 0
+P 3550 13050
+F 0 "#PWR032" H 3550 12800 50  0001 C CNN
+F 1 "GND" H 3550 12900 50  0000 C CNN
+F 2 "" H 3550 13050 60  0000 C CNN
+F 3 "" H 3550 13050 60  0000 C CNN
+	1    3550 13050
+	1    0    0    -1
+$EndComp
+Text Label 2950 12550 0    60   ~ 0
 Vbus
 $Comp
@@
 	2600 12650 3550 12650
 Wire Wire Line
-	2600 12750 3550 12750
-Wire Wire Line
-	3550 12650 3550 12500
-Wire Wire Line
-	3550 12200 3550 12100
-Wire Wire Line
-	3550 12750 3550 12850
-Wire Wire Line
-	2600 13050 3550 13050
-Wire Wire Line
-	3550 13050 3550 13150
-Wire Wire Line
-	2600 13150 3150 13150
+	3250 13850 3250 13700
+Wire Wire Line
+	3250 13400 3250 13300
+Wire Wire Line
+	3550 12650 3550 12750
+Wire Wire Line
+	2600 12950 3550 12950
+Wire Wire Line
+	3550 12950 3550 13050
+Wire Wire Line
+	2600 12550 3150 12550
+Wire Wire Line
+	2600 12750 3000 12750
 Wire Wire Line
 	2600 12850 3000 12850
 Wire Wire Line
-	2600 12950 3000 12950
-Wire Wire Line
-	2600 12550 3000 12550
+	2600 13050 3000 13050
 Wire Wire Line
 	5700 20850 6500 20850
@@
 $EndComp
 Wire Wire Line
-	2600 13250 3350 13250
-Wire Wire Line
-	3350 13250 3350 13350
+	2700 13250 2700 13350
 $Comp
 L GND #PWR091
 U 1 1 566EF91F
-P 3350 13350
-F 0 "#PWR091" H 3350 13100 50  0001 C CNN
-F 1 "GND" H 3350 13200 50  0000 C CNN
-F 2 "" H 3350 13350 60  0000 C CNN
-F 3 "" H 3350 13350 60  0000 C CNN
-	1    3350 13350
+P 2700 13350
+F 0 "#PWR091" H 2700 13100 50  0001 C CNN
+F 1 "GND" H 2700 13200 50  0000 C CNN
+F 2 "" H 2700 13350 60  0000 C CNN
+F 3 "" H 2700 13350 60  0000 C CNN
+	1    2700 13350
 	1    0    0    -1
 $EndComp
@@
 Wire Wire Line
 	1300 21050 1300 20950
+Wire Wire Line
+	2700 13250 2600 13250
+Wire Wire Line
+	2600 13150 3000 13150
+Wire Wire Line
+	3000 13150 3000 13850
+Wire Wire Line
+	3000 13850 3250 13850
 $EndSCHEMATC

Commit message: a
Changed lines of the file:
@@
 Text Label 9700 4200 0    60   ~ 0
 gpio-2
-Text Label 9700 8900 0    60   ~ 0
+Text Label 9700 9300 0    60   ~ 0
 gpio-3
 Text Label 2700 13050 0    60   ~ 0
@@
 	9150 2300 10000 2300
 Wire Wire Line
-	9150 8900 10000 8900
+	9150 9300 10000 9300
 Wire Wire Line
 	9150 4200 10000 4200
@@
 Text Label 9200 8500 0    60   ~ 0
 ~enable~
-Text Label 9200 9100 0    60   ~ 0
+Text Label 9200 4000 0    60   ~ 0
 ~reset~
 Text Label 9200 3800 0    60   ~ 0
 ~sleep~
-Text Label 9200 4000 0    60   ~ 0
+Text Label 9200 9100 0    60   ~ 0
 ~high-current~
 Text Label 9200 6950 0    60   ~ 0
@@
 Text Label 9200 3600 0    60   ~ 0
 hall1
-Text Label 9200 9300 0    60   ~ 0
+Text Label 9200 8900 0    60   ~ 0
 hall2
 Text Label 9200 8100 0    60   ~ 0
@@
 	9150 8500 9500 8500
 Wire Wire Line
-	9150 9100 9500 9100
+	9150 4000 9500 4000
 Wire Wire Line
 	9150 3800 9500 3800
 Wire Wire Line
-	9150 4000 9800 4000
+	9150 9100 9800 9100
 Wire Wire Line
 	9150 6950 9450 6950
@@
 	9150 3600 9450 3600
 Wire Wire Line
-	9150 9300 9450 9300
+	9150 8900 9450 8900
 Wire Wire Line
 	9150 8100 9950 8100

Commit message: Finished routing.
Changed lines of the file:
@@
 Text Label 9800 3200 0    60   ~ 0
 rx-2
-Text Label 9250 7150 0    60   ~ 0
+Text Label 9600 4200 0    60   ~ 0
 gpio-0
 Text Label 9700 9500 0    60   ~ 0
 gpio-1
-Text Label 9700 4200 0    60   ~ 0
+Text Label 9700 9300 0    60   ~ 0
 gpio-2
-Text Label 9700 9300 0    60   ~ 0
+Text Label 9700 7150 0    60   ~ 0
 gpio-3
 Text Label 2700 13050 0    60   ~ 0
@@
 	4550 5900 4100 5900
 Wire Wire Line
-	9600 7150 9150 7150
+	9150 4200 9950 4200
 Wire Wire Line
 	1200 12950 1200 12750
@@
 	9150 2300 10000 2300
 Wire Wire Line
+	9150 7150 10000 7150
+Wire Wire Line
 	9150 9300 10000 9300
 Wire Wire Line
-	9150 4200 10000 4200
-Wire Wire Line
 	9150 9500 10000 9500
