File: electrical/lcu03/stepper-subcircuit.sch (KiCad schematic (older format))
At the start: 12 parts, among them P14 stepper_conn, U8 a4985

Commit message: a
Parts:
- added R45: 100 5%, Resistors_SMD:R_0805, symbol R
Connections:
- wire segments 59 -> 61

Commit message: a
Changed lines of the file:
@@
 AR Path="/5667C1E7/5667C673" Ref="U8"  Part="1"
 AR Path="/56687F5B/5667C673" Ref="U9"  Part="1"
-F 0 "U8" H 4650 4550 60  0000 C CNN
+F 0 "U9" H 4650 4550 60  0000 C CNN
 F 1 "a4985" V 4650 3350 60  0000 C CNN
 F 2 "my-lib:a4985" H 4650 3350 60  0001 C CNN
@@
 AR Path="/5667C1E7/5667C682" Ref="C28"  Part="1"
 AR Path="/56687F5B/5667C682" Ref="C34"  Part="1"
-F 0 "C28" H 3725 2450 50  0000 L CNN
+F 0 "C34" H 3725 2450 50  0000 L CNN
 F 1 "100n" V 3650 2000 50  0000 L CNN
 F 2 "Capacitors_SMD:C_0805" H 3738 2200 50  0001 C CNN
@@
 AR Path="/5667C1E7/5667C68D" Ref="C29"  Part="1"
 AR Path="/56687F5B/5667C68D" Ref="C35"  Part="1"
-F 0 "C29" H 3725 2850 50  0000 L CNN
+F 0 "C35" H 3725 2850 50  0000 L CNN
 F 1 "100n" V 3650 2450 50  0000 L CNN
 F 2 "Capacitors_SMD:C_0805" H 3738 2600 50  0001 C CNN
@@
 AR Path="/5667C1E7/5667C697" Ref="C30"  Part="1"
 AR Path="/56687F5B/5667C697" Ref="C36"  Part="1"
-F 0 "C30" H 3725 3050 50  0000 L CNN
+F 0 "C36" H 3725 3050 50  0000 L CNN
 F 1 "220n" V 3650 2650 50  0000 L CNN
 F 2 "Capacitors_SMD:C_0805" H 3738 2800 50  0001 C CNN
@@
 	3150 2950 3150 3050
 $Comp
-L GND #PWR094
+L GND #PWR92
 U 1 1 5667C6A1
 P 3150 3050
-AR Path="/5667C1E7/5667C6A1" Ref="#PWR094"  Part="1"
-AR Path="/56687F5B/5667C6A1" Ref="#PWR0106"  Part="1"
-F 0 "#PWR0106" H 3150 2800 50  0001 C CNN
+AR Path="/5667C1E7/5667C6A1" Ref="#PWR92"  Part="1"
+AR Path="/56687F5B/5667C6A1" Ref="#PWR104"  Part="1"
+F 0 "#PWR104" H 3150 2800 50  0001 C CNN
 F 1 "GND" H 3150 2900 50  0000 C CNN
 F 2 "" H 3150 3050 50  0000 C CNN
@@
 AR Path="/5667C1E7/5667C6AF" Ref="C27"  Part="1"
 AR Path="/56687F5B/5667C6AF" Ref="C33"  Part="1"
-F 0 "C27" H 3175 4500 50  0000 L CNN
+F 0 "C33" H 3175 4500 50  0000 L CNN
 F 1 "100n" H 3175 4300 50  0000 L CNN
 F 2 "Capacitors_SMD:C_0805" H 3188 4250 50  0001 C CNN
@@
 	3150 4550 3150 4650
 $Comp
-L GND #PWR095
+L GND #PWR93
 U 1 1 5667C6B8
 P 3150 4650
-AR Path="/5667C1E7/5667C6B8" Ref="#PWR095"  Part="1"
-AR Path="/56687F5B/5667C6B8" Ref="#PWR0107"  Part="1"
-F 0 "#PWR0107" H 3150 4400 50  0001 C CNN
+AR Path="/5667C1E7/5667C6B8" Ref="#PWR93"  Part="1"
+AR Path="/56687F5B/5667C6B8" Ref="#PWR105"  Part="1"
+F 0 "#PWR105" H 3150 4400 50  0001 C CNN
 F 1 "GND" H 3150 4500 50  0000 C CNN
 F 2 "" H 3150 4650 50  0000 C CNN
@@
 	5450 4550 5450 4750
 $Comp
-L GND #PWR096
+L GND #PWR96
 U 1 1 5667C6C4
 P 5450 4750
-AR Path="/5667C1E7/5667C6C4" Ref="#PWR096"  Part="1"
-AR Path="/56687F5B/5667C6C4" Ref="#PWR0108"  Part="1"
-F 0 "#PWR0108" H 5450 4500 50  0001 C CNN
+AR Path="/5667C1E7/5667C6C4" Ref="#PWR96"  Part="1"
+AR Path="/56687F5B/5667C6C4" Ref="#PWR108"  Part="1"
+F 0 "#PWR108" H 5450 4500 50  0001 C CNN
 F 1 "GND" H 5450 4600 50  0000 C CNN
 F 2 "" H 5450 4750 50  0000 C CNN
@@
 	4550 4850 4550 5050
 $Comp
-L GND #PWR097
+L GND #PWR95
 U 1 1 5667C6CB
 P 4550 5050
-AR Path="/5667C1E7/5667C6CB" Ref="#PWR097"  Part="1"
-AR Path="/56687F5B/5667C6CB" Ref="#PWR0109"  Part="1"
-F 0 "#PWR0109" H 4550 4800 50  0001 C CNN
+AR Path="/5667C1E7/5667C6CB" Ref="#PWR95"  Part="1"
+AR Path="/56687F5B/5667C6CB" Ref="#PWR107"  Part="1"
+F 0 "#PWR107" H 4550 4800 50  0001 C CNN
 F 1 "GND" H 4550 4900 50  0000 C CNN
 F 2 "" H 4550 5050 50  0000 C CNN
@@
 	4050 3750 2750 3750
 $Comp
-L GND #PWR098
+L GND #PWR91
 U 1 1 5667C6DE
 P 2750 4450
-AR Path="/5667C1E7/5667C6DE" Ref="#PWR098"  Part="1"
-AR Path="/56687F5B/5667C6DE" Ref="#PWR0110"  Part="1"
-F 0 "#PWR0110" H 2750 4200 50  0001 C CNN
+AR Path="/5667C1E7/5667C6DE" Ref="#PWR91"  Part="1"
+AR Path="/56687F5B/5667C6DE" Ref="#PWR103"  Part="1"
+F 0 "#PWR103" H 2750 4200 50  0001 C CNN
 F 1 "GND" H 2750 4300 50  0000 C CNN
 F 2 "" H 2750 4450 50  0000 C CNN
@@
 	7000 4350 7000 4450
 $Comp
-L GND #PWR099
+L GND #PWR98
 U 1 1 5667C6ED
 P 7000 4450
-AR Path="/5667C1E7/5667C6ED" Ref="#PWR099"  Part="1"
-AR Path="/56687F5B/5667C6ED" Ref="#PWR0111"  Part="1"
-F 0 "#PWR0111" H 7000 4200 50  0001 C CNN
+AR Path="/5667C1E7/5667C6ED" Ref="#PWR98"  Part="1"
+AR Path="/56687F5B/5667C6ED" Ref="#PWR110"  Part="1"
+F 0 "#PWR110" H 7000 4200 50  0001 C CNN
 F 1 "GND" H 7000 4300 50  0000 C CNN
 F 2 "" H 7000 4450 50  0000 C CNN
@@
 AR Path="/5667C1E7/5667C6F4" Ref="R39"  Part="1"
 AR Path="/56687F5B/5667C6F4" Ref="R43"  Part="1"
-F 0 "R39" V 8530 3150 40  0000 C CNN
+F 0 "R43" V 8530 3150 40  0000 C CNN
 F 1 "1 5%" V 8457 3151 40  0000 C CNN
 F 2 "Resistors_SMD:R_0805" V 8380 3150 30  0001 C CNN
@@
 AR Path="/5667C1E7/5667C708" Ref="C32"  Part="1"
 AR Path="/56687F5B/5667C708" Ref="C38"  Part="1"
-F 0 "C32" H 7025 4300 50  0000 L CNN
+F 0 "C38" H 7025 4300 50  0000 L CNN
 F 1 "100n" H 7025 4100 50  0000 L CNN
 F 2 "Capacitors_SMD:C_0805" H 7038 4050 50  0001 C CNN
@@
 	8900 3150 8900 3350
 $Comp
-L GND #PWR0100
+L GND #PWR99
 U 1 1 5667C713
 P 8900 3350
-AR Path="/5667C1E7/5667C713" Ref="#PWR0100"  Part="1"
-AR Path="/56687F5B/5667C713" Ref="#PWR0112"  Part="1"
-F 0 "#PWR0112" H 8900 3100 50  0001 C CNN
+AR Path="/5667C1E7/5667C713" Ref="#PWR99"  Part="1"
+AR Path="/56687F5B/5667C713" Ref="#PWR111"  Part="1"
+F 0 "#PWR111" H 8900 3100 50  0001 C CNN
 F 1 "GND" H 8900 3200 50  0000 C CNN
 F 2 "" H 8900 3350 50  0000 C CNN
@@
 AR Path="/5667C1E7/5667C719" Ref="R40"  Part="1"
 AR Path="/56687F5B/5667C719" Ref="R44"  Part="1"
-F 0 "R40" V 8530 3750 40  0000 C CNN
+F 0 "R44" V 8530 3750 40  0000 C CNN
 F 1 "1 5%" V 8457 3751 40  0000 C CNN
 F 2 "Resistors_SMD:R_0805" V 8380 3750 30  0001 C CNN
@@
 	8900 3750 8900 3950
 $Comp
-L GND #PWR0101
+L GND #PWR100
 U 1 1 5667C724
 P 8900 3950
-AR Path="/5667C1E7/5667C724" Ref="#PWR0101"  Part="1"
-AR Path="/56687F5B/5667C724" Ref="#PWR0113"  Part="1"
-F 0 "#PWR0113" H 8900 3700 50  0001 C CNN
+AR Path="/5667C1E7/5667C724" Ref="#PWR100"  Part="1"
+AR Path="/56687F5B/5667C724" Ref="#PWR112"  Part="1"
+F 0 "#PWR112" H 8900 3700 50  0001 C CNN
 F 1 "GND" H 8900 3800 50  0000 C CNN
 F 2 "" H 8900 3950 50  0000 C CNN
@@
 	6100 2350 6100 2550
 $Comp
-L GND #PWR0102
+L GND #PWR97
 U 1 1 5667C72E
 P 6100 2550
-AR Path="/5667C1E7/5667C72E" Ref="#PWR0102"  Part="1"
-AR Path="/56687F5B/5667C72E" Ref="#PWR0114"  Part="1"
-F 0 "#PWR0114" H 6100 2300 50  0001 C CNN
+AR Path="/5667C1E7/5667C72E" Ref="#PWR97"  Part="1"
+AR Path="/56687F5B/5667C72E" Ref="#PWR109"  Part="1"
+F 0 "#PWR109" H 6100 2300 50  0001 C CNN
 F 1 "GND" H 6100 2400 50  0000 C CNN
 F 2 "" H 6100 2550 50  0000 C CNN
@@
 AR Path="/5667C1E7/566C867B" Ref="R37"  Part="1"
 AR Path="/56687F5B/566C867B" Ref="R41"  Part="1"
-F 0 "R37" V 1430 4350 50  0000 C CNN
+F 0 "R41" V 1430 4350 50  0000 C CNN
 F 1 "100 5%" V 1350 4350 50  0000 C CNN
 F 2 "Resistors_SMD:R_0805" V 1280 4350 50  0001 C CNN
@@
 AR Path="/5667C1E7/566C8917" Ref="R38"  Part="1"
 AR Path="/56687F5B/566C8917" Ref="R42"  Part="1"
-F 0 "R38" V 1430 4600 50  0000 C CNN
+F 0 "R42" V 1430 4600 50  0000 C CNN
 F 1 "100 5%" V 1350 4600 50  0000 C CNN
 F 2 "Resistors_SMD:R_0805" V 1280 4600 50  0001 C CNN
@@
 AR Path="/5667C1E7/5668FCA0" Ref="P14"  Part="1"
 AR Path="/56687F5B/5668FCA0" Ref="P15"  Part="1"
-F 0 "P14" H 10100 3850 50  0000 C CNN
+F 0 "P15" H 10100 3850 50  0000 C CNN
 F 1 "stepper_conn" V 10150 3500 50  0000 C CNN
 F 2 "my-lib:JST_B4B-PH-SM4-TB" H 10050 3600 50  0001 C CNN
@@
 	10050 4000 10050 4100
 $Comp
-L GND #PWR0103
+L GND #PWR101
 U 1 1 5668FCAB
 P 10050 4100
-AR Path="/5667C1E7/5668FCAB" Ref="#PWR0103"  Part="1"
-AR Path="/56687F5B/5668FCAB" Ref="#PWR0115"  Part="1"
-F 0 "#PWR0115" H 10050 3850 50  0001 C CNN
+AR Path="/5667C1E7/5668FCAB" Ref="#PWR101"  Part="1"
+AR Path="/56687F5B/5668FCAB" Ref="#PWR113"  Part="1"
+F 0 "#PWR113" H 10050 3850 50  0001 C CNN
 F 1 "GND" H 10050 3950 50  0000 C CNN
 F 2 "" H 10050 4100 60  0000 C CNN
@@
 $EndComp
 $Comp
-L GND #PWR0104
+L GND #PWR102
 U 1 1 5668FCB1
 P 10350 3200
-AR Path="/5667C1E7/5668FCB1" Ref="#PWR0104"  Part="1"
-AR Path="/56687F5B/5668FCB1" Ref="#PWR0116"  Part="1"
-F 0 "#PWR0116" H 10350 2950 50  0001 C CNN
+AR Path="/5667C1E7/5668FCB1" Ref="#PWR102"  Part="1"
+AR Path="/56687F5B/5668FCB1" Ref="#PWR114"  Part="1"
+F 0 "#PWR114" H 10350 2950 50  0001 C CNN
 F 1 "GND" H 10350 3050 50  0000 C CNN
 F 2 "" H 10350 3200 60  0000 C CNN
@@
 AR Path="/5667C1E7/567280CE" Ref="R45"  Part="1"
 AR Path="/56687F5B/567280CE" Ref="R46"  Part="1"
-F 0 "R45" V 2830 4050 50  0000 C CNN
+F 0 "R46" V 2830 4050 50  0000 C CNN
 F 1 "100 5%" V 2750 4050 50  0000 C CNN
 F 2 "Resistors_SMD:R_0805" V 2680 4050 50  0001 C CNN
@@
 AR Path="/5667C1E7/5672F546" Ref="C31"  Part="1"
 AR Path="/56687F5B/5672F546" Ref="C37"  Part="1"
-F 0 "C31" H 3825 4900 50  0000 L CNN
+F 0 "C37" H 3825 4900 50  0000 L CNN
 F 1 "100n" H 3825 4700 50  0000 L CNN
 F 2 "Capacitors_SMD:C_0805" H 3838 4650 50  0001 C CNN
@@
 	3800 4950 3800 5050
 $Comp
-L GND #PWR0105
+L GND #PWR94
 U 1 1 5672F679
 P 3800 5050
-AR Path="/5667C1E7/5672F679" Ref="#PWR0105"  Part="1"
-AR Path="/56687F5B/5672F679" Ref="#PWR0117"  Part="1"
-F 0 "#PWR0117" H 3800 4800 50  0001 C CNN
+AR Path="/5667C1E7/5672F679" Ref="#PWR94"  Part="1"
+AR Path="/56687F5B/5672F679" Ref="#PWR106"  Part="1"
+F 0 "#PWR106" H 3800 4800 50  0001 C CNN
 F 1 "GND" H 3800 4900 50  0000 C CNN
 F 2 "" H 3800 5050 50  0000 C CNN

Commit message: a
Connections:
- net labels added: out1a, out1b, out2a, out2b, rsense1, rsense2
- net labels removed: out1a-1, out1b-1, out2a-1, out2b-1, rsense1-1, rsense2-1
- wire segments 61 -> 59
Other:
- moved on the sheet: C33, R41, R42, R46

Commit message: Replaced linear regulator, changed socket footprints and implemented all improvements from "zzz.txt" file.
Parts:
- P14: footprint my-lib:JST_B4B-PH-SM4-TB -> my-lib:my-JST_B4B-PH-SM4-TB
Changed lines of the file:
@@
 LIBS:m24c02
 LIBS:stepper_conn
+LIBS:my-ncp1117st50t3g
 LIBS:lcu03-cache
 EELAYER 25 0
@@
 	3150 2950 3150 3050
 $Comp
-L GND #PWR097
+L GND #PWR096
 U 1 1 5667C6A1
 P 3150 3050
-AR Path="/5667C1E7/5667C6A1" Ref="#PWR097"  Part="1"
-AR Path="/56687F5B/5667C6A1" Ref="#PWR0109"  Part="1"
-F 0 "#PWR0109" H 3150 2800 50  0001 C CNN
+AR Path="/5667C1E7/5667C6A1" Ref="#PWR096"  Part="1"
+AR Path="/56687F5B/5667C6A1" Ref="#PWR0108"  Part="1"
+F 0 "#PWR0108" H 3150 2800 50  0001 C CNN
 F 1 "GND" H 3150 2900 50  0000 C CNN
 F 2 "" H 3150 3050 50  0000 C CNN
@@
 	2700 4550 2700 4650
 $Comp
-L GND #PWR098
+L GND #PWR097
 U 1 1 5667C6B8
 P 2700 4650
-AR Path="/5667C1E7/5667C6B8" Ref="#PWR098"  Part="1"
-AR Path="/56687F5B/5667C6B8" Ref="#PWR0110"  Part="1"
-F 0 "#PWR0110" H 2700 4400 50  0001 C CNN
+AR Path="/5667C1E7/5667C6B8" Ref="#PWR097"  Part="1"
+AR Path="/56687F5B/5667C6B8" Ref="#PWR0109"  Part="1"
+F 0 "#PWR0109" H 2700 4400 50  0001 C CNN
 F 1 "GND" H 2700 4500 50  0000 C CNN
 F 2 "" H 2700 4650 50  0000 C CNN
@@
 	5450 4550 5450 4750
 $Comp
-L GND #PWR099
+L GND #PWR098
 U 1 1 5667C6C4
 P 5450 4750
-AR Path="/5667C1E7/5667C6C4" Ref="#PWR099"  Part="1"
-AR Path="/56687F5B/5667C6C4" Ref="#PWR0111"  Part="1"
-F 0 "#PWR0111" H 5450 4500 50  0001 C CNN
+AR Path="/5667C1E7/5667C6C4" Ref="#PWR098"  Part="1"
+AR Path="/56687F5B/5667C6C4" Ref="#PWR0110"  Part="1"
+F 0 "#PWR0110" H 5450 4500 50  0001 C CNN
 F 1 "GND" H 5450 4600 50  0000 C CNN
 F 2 "" H 5450 4750 50  0000 C CNN
@@
 	4550 4850 4550 5050
 $Comp
-L GND #PWR0100
+L GND #PWR099
 U 1 1 5667C6CB
 P 4550 5050
-AR Path="/5667C1E7/5667C6CB" Ref="#PWR0100"  Part="1"
-AR Path="/56687F5B/5667C6CB" Ref="#PWR0112"  Part="1"
-F 0 "#PWR0112" H 4550 4800 50  0001 C CNN
+AR Path="/5667C1E7/5667C6CB" Ref="#PWR099"  Part="1"
+AR Path="/56687F5B/5667C6CB" Ref="#PWR0111"  Part="1"
+F 0 "#PWR0111" H 4550 4800 50  0001 C CNN
 F 1 "GND" H 4550 4900 50  0000 C CNN
 F 2 "" H 4550 5050 50  0000 C CNN
@@
 	2300 3750 4050 3750
 $Comp
-L GND #PWR0101
+L GND #PWR0100
 U 1 1 5667C6DE
 P 2300 4450
-AR Path="/5667C1E7/5667C6DE" Ref="#PWR0101"  Part="1"
-AR Path="/56687F5B/5667C6DE" Ref="#PWR0113"  Part="1"
-F 0 "#PWR0113" H 2300 4200 50  0001 C CNN
+AR Path="/5667C1E7/5667C6DE" Ref="#PWR0100"  Part="1"
+AR Path="/56687F5B/5667C6DE" Ref="#PWR0112"  Part="1"
+F 0 "#PWR0112" H 2300 4200 50  0001 C CNN
 F 1 "GND" H 2300 4300 50  0000 C CNN
 F 2 "" H 2300 4450 50  0000 C CNN
@@
 	7000 4350 7000 4450
 $Comp
-L GND #PWR0102
+L GND #PWR0101
 U 1 1 5667C6ED
 P 7000 4450
-AR Path="/5667C1E7/5667C6ED" Ref="#PWR0102"  Part="1"
-AR Path="/56687F5B/5667C6ED" Ref="#PWR0114"  Part="1"
-F 0 "#PWR0114" H 7000 4200 50  0001 C CNN
+AR Path="/5667C1E7/5667C6ED" Ref="#PWR0101"  Part="1"
+AR Path="/56687F5B/5667C6ED" Ref="#PWR0113"  Part="1"
+F 0 "#PWR0113" H 7000 4200 50  0001 C CNN
 F 1 "GND" H 7000 4300 50  0000 C CNN
 F 2 "" H 7000 4450 50  0000 C CNN
@@
 	8900 3150 8900 3350
 $Comp
-L GND #PWR0103
+L GND #PWR0102
 U 1 1 5667C713
 P 8900 3350
-AR Path="/5667C1E7/5667C713" Ref="#PWR0103"  Part="1"
-AR Path="/56687F5B/5667C713" Ref="#PWR0115"  Part="1"
-F 0 "#PWR0115" H 8900 3100 50  0001 C CNN
+AR Path="/5667C1E7/5667C713" Ref="#PWR0102"  Part="1"
+AR Path="/56687F5B/5667C713" Ref="#PWR0114"  Part="1"
+F 0 "#PWR0114" H 8900 3100 50  0001 C CNN
 F 1 "GND" H 8900 3200 50  0000 C CNN
 F 2 "" H 8900 3350 50  0000 C CNN
@@
 	8900 3750 8900 3950
 $Comp
-L GND #PWR0104
+L GND #PWR0103
 U 1 1 5667C724
 P 8900 3950
-AR Path="/5667C1E7/5667C724" Ref="#PWR0104"  Part="1"
-AR Path="/56687F5B/5667C724" Ref="#PWR0116"  Part="1"
-F 0 "#PWR0116" H 8900 3700 50  0001 C CNN
+AR Path="/5667C1E7/5667C724" Ref="#PWR0103"  Part="1"
+AR Path="/56687F5B/5667C724" Ref="#PWR0115"  Part="1"
+F 0 "#PWR0115" H 8900 3700 50  0001 C CNN
 F 1 "GND" H 8900 3800 50  0000 C CNN
 F 2 "" H 8900 3950 50  0000 C CNN
@@
 	6100 2350 6100 2550
 $Comp
-L GND #PWR0105
+L GND #PWR0104
 U 1 1 5667C72E
 P 6100 2550
-AR Path="/5667C1E7/5667C72E" Ref="#PWR0105"  Part="1"
-AR Path="/56687F5B/5667C72E" Ref="#PWR0117"  Part="1"
-F 0 "#PWR0117" H 6100 2300 50  0001 C CNN
+AR Path="/5667C1E7/5667C72E" Ref="#PWR0104"  Part="1"
+AR Path="/56687F5B/5667C72E" Ref="#PWR0116"  Part="1"
+F 0 "#PWR0116" H 6100 2300 50  0001 C CNN
 F 1 "GND" H 6100 2400 50  0000 C CNN
 F 2 "" H 6100 2550 50  0000 C CNN
@@
 F 0 "P15" H 10100 3850 50  0000 C CNN
 F 1 "stepper_conn" V 10150 3500 50  0000 C CNN
-F 2 "my-lib:JST_B4B-PH-SM4-TB" H 10050 3600 50  0001 C CNN
+F 2 "my-lib:my-JST_B4B-PH-SM4-TB" H 10050 3600 50  0001 C CNN
 F 3 "" H 10050 3600 50  0000 C CNN
 	1    10050 3600
@@
 	10050 4000 10050 4100
 $Comp
-L GND #PWR0106
+L GND #PWR0105
 U 1 1 5668FCAB
 P 10050 4100
-AR Path="/5667C1E7/5668FCAB" Ref="#PWR0106"  Part="1"
-AR Path="/56687F5B/5668FCAB" Ref="#PWR0118"  Part="1"
-F 0 "#PWR0118" H 10050 3850 50  0001 C CNN
+AR Path="/5667C1E7/5668FCAB" Ref="#PWR0105"  Part="1"
+AR Path="/56687F5B/5668FCAB" Ref="#PWR0117"  Part="1"
+F 0 "#PWR0117" H 10050 3850 50  0001 C CNN
 F 1 "GND" H 10050 3950 50  0000 C CNN
 F 2 "" H 10050 4100 60  0000 C CNN
@@
 $EndComp
 $Comp
-L GND #PWR0107
+L GND #PWR0106
 U 1 1 5668FCB1
 P 10350 3200
-AR Path="/5667C1E7/5668FCB1" Ref="#PWR0107"  Part="1"
-AR Path="/56687F5B/5668FCB1" Ref="#PWR0119"  Part="1"
-F 0 "#PWR0119" H 10350 2950 50  0001 C CNN
+AR Path="/5667C1E7/5668FCB1" Ref="#PWR0106"  Part="1"
+AR Path="/56687F5B/5668FCB1" Ref="#PWR0118"  Part="1"
+F 0 "#PWR0118" H 10350 2950 50  0001 C CNN
 F 1 "GND" H 10350 3050 50  0000 C CNN
 F 2 "" H 10350 3200 60  0000 C CNN
@@
 	3800 4950 3800 5050
 $Comp
-L GND #PWR0108
+L GND #PWR0107
 U 1 1 5672F679
 P 3800 5050
-AR Path="/5667C1E7/5672F679" Ref="#PWR0108"  Part="1"
-AR Path="/56687F5B/5672F679" Ref="#PWR0120"  Part="1"
-F 0 "#PWR0120" H 3800 4800 50  0001 C CNN
+AR Path="/5667C1E7/5672F679" Ref="#PWR0107"  Part="1"
+AR Path="/56687F5B/5672F679" Ref="#PWR0119"  Part="1"
+F 0 "#PWR0119" H 3800 4800 50  0001 C CNN
 F 1 "GND" H 3800 4900 50  0000 C CNN
 F 2 "" H 3800 5050 50  0000 C CNN
