File: controller-em-tests/lm317-vs/lm317-vs.kicad_pcb (KiCad board)
At the start: 2 copper layers, 47 x 19 mm, 13 parts, among them P1 in-15v, P2 gnd, P3 out-12v, P4 gnd, U1 LM317EMP

Commit message: a
Parts:
- R1: value 6k8 -> 820R
- R2: value 820R -> 6k8
Changed lines of the file:
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@@
     (links 20)
     (no_connects 0)
-    (area 141.924999 96.924999 189.417858 116.075001)
+    (area 141.924999 96.924999 189.075001 116.075001)
     (thickness 1.6)
     (drawings 4)
@@
   )
   (setup
-    (last_trace_width 1.2)
+    (last_trace_width 0.25)
     (user_trace_width 0.4)
     (user_trace_width 0.5)
@@
     (pad_to_mask_clearance 0.2)
     (aux_axis_origin 0 0)
-    (visible_elements FFFFFF7F)
+    (visible_elements 7FFFFFFF)
     (pcbplotparams
       (layerselection 0x00030_80000001)
@@
       (effects (font (size 1 1) (thickness 0.15)))
     )
-    (fp_text value 4u7 (at 0 2.1 270) (layer F.Fab)
+    (fp_text value 4u7 (at -0.25 0.25 270) (layer F.Fab)
       (effects (font (size 1 1) (thickness 0.15)))
     )
@@
       (effects (font (size 1 1) (thickness 0.15)))
     )
-    (fp_text value 100n (at 0 2.1 270) (layer F.Fab)
+    (fp_text value 100n (at -0.25 0.5 270) (layer F.Fab)
       (effects (font (size 1 1) (thickness 0.15)))
     )
@@
       (effects (font (size 1 1) (thickness 0.15)))
     )
-    (fp_text value 100n (at 0 2.1 90) (layer F.Fab)
+    (fp_text value 100n (at -0.05 0.15 90) (layer F.Fab)
       (effects (font (size 1 1) (thickness 0.15)))
     )
@@
       (effects (font (size 1 1) (thickness 0.15)))
     )
-    (fp_text value 6k8 (at 0 2.1 90) (layer F.Fab)
+    (fp_text value 820R (at 0 0.5 90) (layer F.Fab)
       (effects (font (size 1 1) (thickness 0.15)))
     )
@@
       (effects (font (size 1 1) (thickness 0.15)))
     )
-    (fp_text value 820R (at 0 2.1 90) (layer F.Fab)
+    (fp_text value 6k8 (at -0.05 0.15 90) (layer F.Fab)
       (effects (font (size 1 1) (thickness 0.15)))
     )
@@
   (segment (start 145.85 103.8) (end 150.05 108) (width 1.2) (layer F.Cu) (net 1))
   (segment (start 150.05 108) (end 152.25 108) (width 1.2) (layer F.Cu) (net 1))
-  (segment (start 179.25 108.5) (end 179.5 108.5) (width 1.2) (layer F.Cu) (net 2) (status C00000))
-  (segment (start 179.5 108.5) (end 182 111) (width 1.2) (layer F.Cu) (net 2) (status 400000))
-  (segment (start 182 111) (end 186 111) (width 1.2) (layer F.Cu) (net 2) (status 800000))
+  (segment (start 179.25 108.5) (end 179.5 108.5) (width 1.2) (layer F.Cu) (net 2))
+  (segment (start 179.5 108.5) (end 182 111) (width 1.2) (layer F.Cu) (net 2))
+  (segment (start 182 111) (end 186 111) (width 1.2) (layer F.Cu) (net 2))
   (segment (start 154.5 110.5) (end 154.5 114.5) (width 0.8) (layer F.Cu) (net 2))
   (segment (start 172 114) (end 172 108) (width 0.8) (layer F.Cu) (net 2))
@@
   (segment (start 154.4 102.75) (end 154.5 102.75) (width 0.8) (layer F.Cu) (net 3))
   (segment (start 149.85 105.2) (end 151.85 105.2) (width 1.2) (layer F.Cu) (net 3))
-  (segment (start 179.25 105) (end 180 105) (width 1.2) (layer F.Cu) (net 4) (status 400000))
-  (segment (start 183 102) (end 186 102) (width 1.2) (layer F.Cu) (net 4) (status 800000))
+  (segment (start 179.25 105) (end 180 105) (width 1.2) (layer F.Cu) (net 4))
+  (segment (start 183 102) (end 186 102) (width 1.2) (layer F.Cu) (net 4))
   (segment (start 180 105) (end 183 102) (width 1.2) (layer F.Cu) (net 4))
   (segment (start 174 105.5) (end 176.55 105.5) (width 0.8) (layer F.Cu) (net 4))
