File: controller-em-tests/lm317-vs/lm317-vs.sch (KiCad schematic (older format))
At the start: 13 parts, among them P1 in-15v, P2 gnd, P3 out-12v, P4 gnd, U1 LM317EMP

Commit message: a
Parts:
- R1: value 6k8 -> 820R
- R2: value 820R -> 6k8
Changed lines of the file:
@@
 LIBS:contrib
 LIBS:valves
+LIBS:lm317-vs-cache
 EELAYER 25 0
 EELAYER END
@@
 P 6000 3350
 F 0 "R1" V 6080 3350 50  0000 C CNN
-F 1 "6k8" V 6000 3350 50  0000 C CNN
+F 1 "820R" V 6000 3350 50  0000 C CNN
 F 2 "Capacitors_SMD:C_0805_HandSoldering" V 5930 3350 50  0001 C CNN
 F 3 "" H 6000 3350 50  0000 C CNN
@@
 P 6000 4000
 F 0 "R2" V 6080 4000 50  0000 C CNN
-F 1 "820R" V 6000 4000 50  0000 C CNN
+F 1 "6k8" V 6000 4000 50  0000 C CNN
 F 2 "Capacitors_SMD:C_0805_HandSoldering" V 5930 4000 50  0001 C CNN
 F 3 "" H 6000 4000 50  0000 C CNN
